File: pcie_power.sch (KiCad schematic (older format))
At the start: 24 parts, among them U1 PCIexpress_x4, U2 PCIexpress_x8

Commit message: Switch x8 connector for x4. Add pours and edge cuts
Parts:
- U2: value PCIexpress_x8 -> PCIexpress_x4; footprint Connector_PCBEdge:BUS_PCIexpress_x8 -> Connector_PCBEdge:BUS_PCIexpress_x4; symbol PCIexpress_edge:PCIexpress_x8 -> PCIexpress_edge:PCIexpress_x4
Changed lines of the file:
@@
 $EndComp
 $Comp
-L PCIexpress_edge:PCIexpress_x8 U?
+L PCIexpress_edge:PCIexpress_x4 U?
 U 1 1 5AFB1F39
 P 3450 4500
@@
 AR Path="/5AFB1ECB/5AFB1F39" Ref="U2"  Part="1"
 F 0 "U2" H 4150 4790 60  0000 C CNN
-F 1 "PCIexpress_x8" H 4150 4684 60  0000 C CNN
-F 2 "Connector_PCBEdge:BUS_PCIexpress_x8" H 3450 4500 50  0001 C CNN
+F 1 "PCIexpress_x4" H 4150 4684 60  0000 C CNN
+F 2 "Connector_PCBEdge:BUS_PCIexpress_x4" H 3450 4500 50  0001 C CNN
 F 3 "" H 3450 4500 50  0001 C CNN
 	1    3450 4500
